File: PCAL9539A Breakout/PCAL9539A Breakout.kicad_pcb (KiCad board)
At the start: 2 copper layers, 26.4 x 34 mm, 25 parts, among them J1 Conn_01x06, J2 Conn_01x10, J3 Conn_01x10, U1 PCAL9539A

Commit message: Finished cleanup, silk
Parts:
- added REF**: KiCad-Logo2_5mm_SilkScreen, Symbol:KiCad-Logo2_5mm_SilkScreen, B.Cu at (145.5, 120.1)
- added REF**: OSHW-Logo_5.7x6mm_SilkScreen, Symbol:OSHW-Logo_5.7x6mm_SilkScreen, B.Cu at (145.8, 109.0)
Other:
- board text added: "00"
- board text added: "00: 0x74 01: 0x75 10: 0x76 11: 0x77"
- board text added: "01"
- board text added: "02"
- board text added: "03"
- board text added: "04"
- board text added: "05"
- board text added: "06"
- board text added: "07"
- board text added: "10"
- board text added: "11"
- board text added: "12"
- board text added: "13"
- board text added: "14"
- board text added: "15"
- board text added: "16"
- board text added: "17"
- board text added: "3V3"
- board text added: "BLU"
- board text added: "BY HAPPY LITTLE PCBS"
- board text added: "GND"
- board text added: "GRN"
- board text added: "INT"
- board text added: "P00"
- board text added: "P01"
- board text added: "P02"
- board text added: "PCAL9539A BREAKOUT"
- board text added: "RED"
- board text added: "REV 1"
- board text added: "RST"
- board text added: "SCL"
- board text added: "SDA"
- board text added: "github.com/akowalczyk18/PCAL9539A-Breakout"
